Commit message: Color added

File: my_bot/urdf/myfirst.urdf (robot description, URDF)
Before this commit: robot my_bot, 1 links, 0 joints
Links:
- added link castor; visual sphere radius=0.1
- added link left_wheel; visual cylinder length=0.05 radius=0.12
- added link right_wheel; visual cylinder length=0.05 radius=0.12
- link base_link: geometry visual box size=0.6 0.2 0.1
Joints:
- added joint base_castor: type fixed, parent base_link, child castor, origin xyz=-0.19 0.0 -0.05
- added joint base_leftwheel: type fixed, parent base_link, child left_wheel, origin xyz=0.2 0.16 0.0
- added joint base_rightwheel: type fixed, parent base_link, child right_wheel, origin xyz=0.2 -0.16 0.0
